Commit message: Re-organize files and add two easier environments

File: urdf/decor_easy.urdf (robot description, URDF)
Before this commit: robot decor, 4 links, 3 joints
Links:
- link decor_base: geometry collision box size=0.85 2 0.1; visual box size=0.85 2 0.1
- link l_decor_one: geometry collision box size=0.85 2 0.1; visual box size=0.85 2 0.1
- link l_decor_three: geometry collision box size=0.3 0.6 0.1; visual box size=0.3 0.6 0.1
- link l_decor_two: geometry collision box size=0.3 0.6 0.1; visual box size=0.3 0.6 0.1

File: urdf/decor_very_easy.urdf (robot description, URDF)
Before this commit: robot decor, 4 links, 3 joints
Links:
- link decor_base: geometry collision box size=0.85 2 0.1; visual box size=0.85 2 0.1
- link l_decor_one: geometry collision box size=0.85 2 0.1; visual box size=0.85 2 0.1
- link l_decor_three: geometry collision box size=0.3 0.5 0.1; visual box size=0.3 0.5 0.1
- link l_decor_two: geometry collision box size=0.3 0.5 0.1; visual box size=0.3 0.5 0.1

File: urdf/object.urdf (robot description, URDF)
Before this commit: robot object, 5 links, 4 joints
Links:
- removed link l_object_four
- link l_object_three: mass None -> 1.0; geometry collision box size=0.6 0.1 0.1; visual box size=0.6 0.1 0.1
Joints:
- removed joint j_object_four
- joint j_object_three: origin xyz=0 0.65 0.35 -> xyz=0 0 0.25
