Commit message: Remove collision and inertial descriptions of green ends

File: urdf/object.urdf (robot description, URDF)
Before this commit: robot object, 5 links, 4 joints
Links:
- link l_object_four: mass 1.0 -> None; geometry visual box size=0.01 0.01 0.01
- link l_object_three: mass 1.0 -> None; geometry visual box size=0.01 0.01 0.01

Commit message: Update installation script

File: urdf/object.urdf (robot description, URDF)
Before this commit: robot object, 4 links, 3 joints
Links:
- added link l_object_four, mass 1.0; collision box size=0.1 0.6 0.1; visual box size=0.1 0.6 0.1
Joints:
- added joint j_object_four: type fixed, parent base_link, child l_object_four, origin xyz=0 0 0.25
