Commit message: Update urdf files by adding fixed fake joints

File: urdf/decor.urdf (robot description, URDF)
Before this commit: robot decor, 4 links, 3 joints
Links:
- link decor_base: geometry collision box size=0.85 2 0.1; visual box size=0.85 2 0.1
- link l_decor_one: geometry collision box size=0.85 2 0.1; visual box size=0.85 2 0.1
- link l_decor_three: geometry collision box size=0.3 0.6 0.1; visual box size=0.3 0.6 0.1
- link l_decor_two: geometry collision box size=0.3 0.6 0.1; visual box size=0.3 0.6 0.1

Commit message: Remove inertial data in URDF

File: urdf/decor.urdf (robot description, URDF)
Before this commit: robot decor, 4 links, 3 joints
Links:
- link decor_base: mass 1.0 -> None
- link l_decor_one: mass 1.0 -> None
- link l_decor_three: mass 1.0 -> None
- link l_decor_two: mass 1.0 -> None

File: urdf/decor_easy.urdf (robot description, URDF)
Before this commit: robot decor, 4 links, 3 joints
Links:
- link decor_base: mass 1.0 -> None
- link l_decor_one: mass 1.0 -> None
- link l_decor_three: mass 1.0 -> None
- link l_decor_two: mass 1.0 -> None

File: urdf/decor_very_easy.urdf (robot description, URDF)
Before this commit: robot decor, 4 links, 3 joints
Links:
- link decor_base: mass 1.0 -> None
- link l_decor_three: mass 1.0 -> None
- link l_decor_two: mass 1.0 -> None

Commit message: Enhance URDF decor files: bigger, green and transparent

File: urdf/decor.urdf (robot description, URDF)
Before this commit: robot decor, 4 links, 3 joints
Links:
- link decor_base: geometry collision box size=1.42 3 0.1; visual box size=1.42 3 0.1
- link l_decor_one: geometry collision box size=1.42 3 0.1; visual box size=1.42 3 0.1
- link l_decor_three: geometry collision box size=0.159 1.2 0.1; visual box size=0.159 1.2 0.1
- link l_decor_two: geometry collision box size=0.159 1.2 0.1; visual box size=0.159 1.2 0.1

File: urdf/decor_easy.urdf (robot description, URDF)
Before this commit: robot decor, 4 links, 3 joints
Links:
- link decor_base: geometry collision box size=1.35 3 0.1; visual box size=1.35 3 0.1
- link l_decor_one: geometry collision box size=1.35 3 0.1; visual box size=1.35 3 0.1
- link l_decor_three: geometry collision box size=0.299 1.1 0.1; visual box size=0.299 1.1 0.1
- link l_decor_two: geometry collision box size=0.299 1.1 0.1; visual box size=0.299 1.1 0.1

File: urdf/decor_very_easy.urdf (robot description, URDF)
Before this commit: robot decor, 4 links, 3 joints
Links:
- link decor_base: geometry collision box size=1.35 3 0.1; visual box size=1.35 3 0.1
- link l_decor_one: geometry collision box size=1.35 3 0.1; visual box size=1.35 3 0.1
- link l_decor_three: geometry collision box size=0.299 1 0.1; visual box size=0.299 1 0.1
- link l_decor_two: geometry collision box size=0.299 1 0.1; visual box size=0.299 1 0.1

Commit message: Add scripts, update decor

File: urdf/decor.urdf (robot description, URDF)
Before this commit: robot decor, 4 links, 3 joints
Links:
- link l_decor_one: mass None -> 1.0
- link l_decor_three: mass None -> 1.0
- link l_decor_two: mass None -> 1.0
Joints:
- joint j_decor_one: origin xyz=0 0 0 rpy=0 0 0 -> xyz=0 0 0
- joint j_decor_three: origin xyz=0 0 0 rpy=0 0 0 -> xyz=0 0 0; parent l_decor_two -> decor_base
- joint j_decor_two: origin xyz=0 0 0 rpy=0 0 0 -> xyz=0 0 0; parent l_decor_one -> decor_base
